File: Actuation/Brushless DC Motor/BH67172NUX.sch (EAGLE design)
At the start: 4 parts, among them IC1 BH67172NUX, IC2 BH67172NUX

Commit message: minor update OSHW logo
Parts:
- added GOLD_ORB_SM1: OSHWLOGO_REF_SM, bfl:OSHWLOGO_REF_SM
Changed lines of the file:
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@@
 <part name="+3V1" library="supply1" deviceset="+3V3" device=""/>
 <part name="+3V2" library="supply1" deviceset="+3V3" device=""/>
+<part name="GOLD_ORB_SM1" library="bfl" deviceset="OSHWLOGO" device="_REF_SM"/>
 </parts>
 <sheets>
@@
 <instance part="+3V1" gate="G$1" x="78.74" y="83.82"/>
 <instance part="+3V2" gate="G$1" x="78.74" y="50.8"/>
+<instance part="GOLD_ORB_SM1" gate="G$1" x="132.08" y="76.2"/>
 </instances>
 <busses>
