File: Development Boards/2530EV/CC2530EV.sch (EAGLE design)
At the start: 42 parts, among them CON1 CC_DEBUGGER, IC1 CC2530, IC2 FT230XQ, IC3 TPS732XX, Q1 32MHz

Commit message: Added CC2530EV reference design; added PDF schematics
Parts:
- removed +3.3V, GND: (no value), con-lstb:MA03-1
- removed B1: 2450BM15A0002SLIM, johanson-technology:2450BM15A0002SLIM
- removed CON1: CC_DEBUGGER, con-3m:2510-
- removed IC1: CC2530, chipcon-ti-v2:CC2530
- removed IC2: FT230XQ, ftdichip:FT230XQ
- removed IC3: TPS732XX, TPS732xx:TPS732XX
- removed J1: (no value), con-lstb:MA05-2
- removed L1: PTC 1A, resistor:L-EUL0603K
- removed LCD3310: (no value), con-lsta:FE05-2
- removed LED1, LED2, LED3, LED4: (no value), led:LEDCHIP-LED0805
- removed PORT0, PORT1: (no value), con-lstb:MA10-1
- removed Q1: 32MHz, crystal:FA-128
- removed R10, R11, R2, R5: 0, resistor:R-EU_R0603K
- removed R3, R4: 10k, resistor:R-EU_R0603K
- removed R6, R7, R8, R9: 470, resistor:R-EU_R0603K
- removed S1: BUTTON1, switch-alco:ALCOSWITCH-SMD
- removed S2: RESET, switch-alco:ALCOSWITCH-SMD
- removed USB: USB-MICRO-AB, con-usb-2:USB-OTG_SHIELD
- added C10, C12: 2u2, resistor:C-EUC0402
- added C11: 100n, resistor:C-EUC0402
- added C13, C14: 27p, resistor:C-EUC0402
- added JP1, JP2: (no value), pinhead:PINHD-1X8
- added JP3: (no value), pinhead:PINHD-1X2
- added JP4: (no value), pinhead:PINHD-1X5
- added U$1: CC2530, chipcon-ti-v2:CC2530
- added U$2: 24530BM15A0002, 24530BM15A0002:24530BM15A0002
- added U$3: TPS732XX, TPS732xx:TPS732XX
- added U$4: XTAL32M, abm_osc:XTAL32M
- added U$5: PUSH_BOT, push_botton:PUSH_BOT
- C1, C2: value 27p -> 100n; device resistor:C-EUC0603K -> resistor:C-EUC0402
- C3: value 1u -> 100n; device resistor:C-EUC0603K -> resistor:C-EUC0402
- C4: value 10u -> 100n; device resistor:C-EUC0603K -> resistor:C-EUC0402
- C5, C7: device resistor:C-EUC0603K -> resistor:C-EUC0402
- C6, C9: value 2u2 -> 100n; device resistor:C-EUC0603K -> resistor:C-EUC0402
- C8: value 100n -> 1u; device resistor:C-EUC0603K -> resistor:C-EUC0402
- L-BEAD: value 40ohm 550mA -> L-BEAD; device resistor:L-EUL0603K -> L-Bead:L-BEAD
- R1: value 56k -> 56K; device resistor:R-EU_R0603K -> resistor:R-EU_R0402
Connections:
- removed net +3V3: +3.3V.1, +3.3V.2, +3.3V.3, C9.1, CON1-2.KL, CON1-9.KL, IC1P.DVDD1, IC1P.DVDD2, IC3.OUT, L-BEAD.1, LCD3310.1, PORT0.1, PORT1.1, R3.2, S1.S, S1.S1
- removed net +3V3A: IC1P.AVDD1, IC1P.AVDD2, IC1P.AVDD3, IC1P.AVDD4, IC1P.AVDD5, IC1P.AVDD6, L-BEAD.2
- removed net +5V: C4.1, C6.1, C7.1, IC2.VCC, IC3.EN, IC3.IN, L1.1
- removed net 0V: B1.GND@1, B1.GND@2, B1.GND@3, C1.2, C2.2, C3.2, C4.2, C5.2, C6.2, C7.2, C8.2, C9.2, CON1-1.KL, GND.1, GND.2, GND.3, IC1P.GND-TP, IC1P.GND@1, IC1P.GND@2, IC1P.GND@3, IC1P.GND@4, IC2.GND, IC2.GND@1, IC3.GND, LCD3310.2, LED1.C, LED2.C, LED3.C, LED4.C, PORT0.2, PORT1.2, R1.1, R2.1, R4.1, R5.2, S2.P, S2.P1, USB.GND, USB.GND@1, USB.GND@2, USB.GND@3, USB.GND@4, USB.ID
- removed net BUTTON1: J1.2, R4.2, S1.P, S1.P1
- removed net DM: IC2.USBDM, USB.D-
- removed net DP: IC2.USBDP, USB.D+
- removed net LCD_CS: IC1S.P1.2, LCD3310.10, PORT1.5
- removed net LCD_D/!C: IC1S.P1.3, LCD3310.6, PORT1.6
- removed net LED1: J1.4, R6.2
- removed net LED2: J1.6, R7.2
- removed net LED3: J1.8, R8.2
- removed net LED4: J1.10, R9.2
- removed net MISO: IC1S.P1.7, PORT1.10
- removed net MOSI: IC1S.P1.6, LCD3310.8, PORT1.9
- removed net N$5: IC1S.RBIAS, R1.2
- removed net P0_0: IC1S.P0.0, PORT0.3
- removed net P0_1: IC1S.P0.1, J1.1, PORT0.4
- removed net P0_2: IC1S.P0.2, PORT0.5, R10.1
- removed net P0_3: IC1S.P0.3, PORT0.6, R11.1
- removed net P0_4: IC1S.P0.4, PORT0.7
- removed net P0_5: IC1S.P0.5, PORT0.8
- removed net P0_6: IC1S.P0.6, PORT0.9
- removed net P0_7: IC1S.P0.7, PORT0.10
- removed net P1_0: IC1S.P1.0, J1.3, PORT1.3
- removed net P1_1: IC1S.P1.1, J1.5, PORT1.4
- removed net P1_4: IC1S.P1.4, J1.7, PORT1.7
- removed net P2_0: IC1S.P2.0, J1.9
- removed net RFN: B1.BAL@1, IC1S.RF-N
- removed net RFP: B1.BAL@2, IC1S.RF-P
- removed net RXD: IC2.RXD, R11.2
- removed net SCLK: IC1S.P1.5, LCD3310.9, PORT1.8
- removed net TXD: IC2.TXD, R10.2
- removed net VIO: C5.1, IC2.!RESET, IC2.3V3OUT, IC2.VCCIO
- new net GND: C1.2, C10.2, C11.2, C12.2, C13.2, C14.2, C2.2, C3.2, C4.2, C5.2, C6.2, C7.2, C8.2, C9.2, JP3.1, JP4.1, R1.1, U$1P.GND-TP, U$1P.GND@1, U$1P.GND@2, U$1P.GND@3, U$1P.GND@4, U$2.GND@1, U$2.GND@2, U$2.GND@3, U$3.GND, U$4.2, U$4.4, U$5.P$2
- new net N$13: JP1.5, U$1S.P0.3
- new net N$14: JP1.6, U$1S.P0.2
- new net N$15: JP1.7, U$1S.P0.1
- new net N$16: JP1.8, U$1S.P0.0
- new net N$17: JP2.1, U$1S.P1.0
- new net N$18: JP2.2, U$1S.P1.1
- new net N$19: JP2.3, U$1S.P1.2
- new net N$20: JP2.4, U$1S.P1.3
- new net N$21: JP2.5, U$1S.P1.4
- new net N$22: JP2.6, U$1S.P1.5
- new net N$23: JP2.7, U$1S.P1.6
- new net N$24: JP2.8, U$1S.P1.7
- new net TX: U$2.UNBAL
- new net V+: C11.1, C12.1, JP3.2, U$3.EN, U$3.IN
- new net VCC: C3.1, C4.1, C5.1, C6.1, C7.1, L-BEAD.2, U$1P.AVDD1, U$1P.AVDD2, U$1P.AVDD3, U$1P.AVDD4, U$1P.AVDD5, U$1P.AVDD6
- new net VDD: C1.1, C10.1, C2.1, JP4.2, L-BEAD.1, U$1P.DVDD1, U$1P.DVDD2, U$3.OUT
- net DBG_DC: now also JP4.4, U$1S.P2.2; no longer CON1-3.KL, IC1S.P2.2
- net DBG_DD: now also JP4.3, U$1S.P2.1; no longer CON1-4.KL, IC1S.P2.1
- net N$1: now also C8.1, U$1P.DCOUPL; no longer C3.1, IC1P.DCOUPL
- net N$10: now also JP1.2, U$1S.P0.6; no longer LED2.A, R7.1
- net N$11: now also JP1.3, U$1S.P0.5; no longer LED3.A, R8.1
- net N$12: now also JP1.4, U$1S.P0.4; no longer LED4.A, R9.1
- net N$2: now also R1.2, U$1S.RBIAS; no longer L1.2, USB.VBUS
- net N$3: now also U$1S.RF-P, U$2.BAL1; no longer C2.1, IC1S.OSC-Q1, Q1.3
- net N$4: now also U$1S.RF-N, U$2.BAL2; no longer C1.1, IC1S.OSC-Q2, Q1.1
- net N$6: now also C9.1, U$3.NR; no longer B1.UNBAL, R5.1
- net N$7: now also C14.1, U$1S.OSC-Q2, U$4.1; no longer IC2.CBUS3, R2.2
- net N$8: now also C13.1, U$1S.OSC-Q1, U$4.3; no longer C8.1, IC3.NR
- net N$9: now also JP1.1, U$1S.P0.7; no longer LED1.A, R6.1
- net RESET: now also JP4.5, U$1S.RESET, U$5.P$1; no longer CON1-7.KL, IC1S.RESET, LCD3310.5, R3.1, S2.S, S2.S1
Other:
- note added: "Debugger"
- note added: "Regulaor 200 mA not miniaturized"
- note added: "SMAC Project - CC2530EV Reference Design"
- note added: "Supply"
- note removed: "ANTENNA"
- note removed: "JUMPER J1 OFF: BUTTON/LEDS DISCONNECTED FROM CC2530"
- note removed: "JUMPER J1 ON: BUTTON/LEDS CONNECTED TO CC2530"
- note removed: "OLIMEX-LCD3310 SPI INTERFACE"
- note removed: "P0 & P1 EXTENSION HEADERS"
- note removed: "PUSH BUTTON & LEDS"
- note removed: "REGULATOR 200mA NOT MINIATURIZED"
- note removed: "REMOVE 0 OHM TO USE P0_2 AND P0_3"
- note removed: "RESET PUSH BUTTON"
- note removed: "SMAC Project - SMAC-2530 Reference Design"
- note removed: "USB TO SERIAL CONVERTER"
- note removed: "USB/SERIAL CONVERTER IS ENABLED WHEN R10 & R11 POPULATED"
- note removed: "WIRELESS MICROCONTROLLER + CC-DEBUGGER INTERFACE + POWER HEADERS"
- moved on the sheet: C1, C2, C3, C4, C5, C6, C7, C8, C9, R1
