File: Development-Boards/SMAC-2530/SMAC-2530.brd (EAGLE design)
At the start: 62.6 x 57.5 mm, 42 parts, among them CON1 CC_DEBUGGER, IC1 CC2530, IC2 FT230XQ, IC3 TPS732XX, Q1 32MHz

Commit message: SMAC-2530 release v1.1, better antenna grounding, removed R0 jumper
Parts:
- removed R5: 0, resistor:R0603K
Connections:
- removed net N$6: B1.1, R5.1
- net 0V: now also B1.1; no longer R5.2
Routing:
- net 0V: track 52.4 -> 55.4 mm, vias 2 -> 13
- net N$6: track 1.28 -> 0.00 mm
Other:
- board text added: "DO NOT ROUTE ANTENNA TO 0V!"
- board text added: "SMAC-2530 DEVELOPMENT BOARD v1.1"
- board text removed: "SMAC-2530 DEVELOPMENT BOARD v1.0"
Changed lines of the file:
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@@
 <layer number="109" name="fp9" color="7" fill="1" visible="no" active="yes"/>
 <layer number="110" name="fp0" color="7" fill="1" visible="no" active="yes"/>
-<layer number="111" name="LPC17xx" color="7" fill="1" visible="yes" active="yes"/>
-<layer number="116" name="Patch_BOT" color="9" fill="4" visible="yes" active="yes"/>
+<layer number="111" name="LPC17xx" color="7" fill="1" visible="no" active="yes"/>
+<layer number="116" name="Patch_BOT" color="9" fill="4" visible="no" active="yes"/>
 <layer number="121" name="_tsilk" color="7" fill="1" visible="no" active="yes"/>
 <layer number="122" name="_bsilk" color="7" fill="1" visible="no" active="yes"/>
@@
 <layer number="144" name="Drill_legend" color="7" fill="1" visible="no" active="yes"/>
 <layer number="151" name="HeatSink" color="7" fill="1" visible="no" active="yes"/>
-<layer number="199" name="Contour" color="7" fill="1" visible="yes" active="yes"/>
+<layer number="199" name="Contour" color="7" fill="1" visible="no" active="yes"/>
 <layer number="200" name="200bmp" color="7" fill="1" visible="no" active="yes"/>
 <layer number="201" name="201bmp" color="2" fill="10" visible="no" active="yes"/>
@@
 <wire x1="62.5" y1="14.6" x2="59.7" y2="14.6" width="0.254" layer="21"/>
 <wire x1="62.5" y1="14.6" x2="62.5" y2="17.4" width="0.254" layer="21"/>
-<text x="24.9" y="15.5" size="1.27" layer="21" font="vector">SMAC-2530 DEVELOPMENT BOARD v1.0</text>
+<text x="24.9" y="15.5" size="1.27" layer="21" font="vector">SMAC-2530 DEVELOPMENT BOARD v1.1</text>
 <text x="73.2" y="40.6" size="1.27" layer="21" font="vector" rot="R90">CC-BY-SA 3.0</text>
+<text x="64.1" y="35.5" size="0.8128" layer="49" font="vector" rot="R90">DO NOT ROUTE ANTENNA TO 0V!</text>
 </plain>
 <attributes>
@@
 <attribute name="VALUE" x="61.368" y="47.289" size="0.8128" layer="27" rot="R270"/>
 </element>
-<element name="R5" library="resistor" package="R0603K" value="0" x="63.1" y="42.4" smashed="yes">
-<attribute name="NAME" x="62.711" y="43.089" size="0.8128" layer="25"/>
-<attribute name="VALUE" x="62.911" y="40.868" size="0.8128" layer="27"/>
-</element>
 <element name="LCD3310" library="con-lsta" package="FE05-2" value="" x="43.18" y="32.258" smashed="yes" rot="R180">
 <attribute name="OC_NEWARK" value="unknown" x="43.18" y="32.258" size="1.778" layer="27" rot="R180" display="off"/>
@@
 <contactref element="B1" pad="6"/>
 <contactref element="C3" pad="2"/>
-<contactref element="R5" pad="2"/>
 <contactref element="USB" pad="GND@4"/>
 <contactref element="USB" pad="GND@1"/>
@@
 <wire x1="64.911" y1="40.128" x2="64.911" y2="40.178" width="0.2032" layer="1"/>
 <wire x1="64.911" y1="40.328" x2="64.839" y2="40.4" width="0.2032" layer="1"/>
-<wire x1="64.839" y1="40.4" x2="64.1" y2="40.4" width="0.2032" layer="1"/>
+<wire x1="64.839" y1="40.4" x2="64.1" y2="40.4" width="0.254" layer="1"/>
 <via x="64.1" y="40.4" extent="1-16" drill="0.254"/>
-<wire x1="60.5" y1="41.975" x2="60.5" y2="41.2" width="0.2032" layer="1"/>
-<wire x1="60.5" y1="41.2" x2="60.5" y2="40.425" width="0.2032" layer="1"/>
+<wire x1="60.5" y1="41.975" x2="60.5" y2="41.2" width="0.254" layer="1"/>
+<wire x1="60.5" y1="41.2" x2="60.5" y2="40.425" width="0.254" layer="1"/>
 <wire x1="61.15" y1="40.425" x2="60.5" y2="40.425" width="0.2032" layer="1"/>
 <via x="60.5" y="41.2" extent="1-16" drill="0.254"/>
@@
 <contactref element="GND" pad="1"/>
 <contactref element="GND" pad="2"/>
-<wire x1="64.911" y1="42.428" x2="63.978" y2="42.428" width="0.2032" layer="1"/>
-<wire x1="63.978" y1="42.428" x2="63.95" y2="42.4" width="0.2032" layer="1"/>
 <wire x1="52.45" y1="41.95" x2="54.65" y2="41.95" width="0.254" layer="1"/>
 <wire x1="54.65" y1="41.95" x2="55.4" y2="41.2" width="0.254" layer="1"/>
@@
 <vertex x="11.7" y="61.1"/>
 <vertex x="64.3" y="61.1"/>
-<vertex x="64.3" y="44.8"/>
-<vertex x="57.6" y="44.8"/>
+<vertex x="64.3" y="43.1"/>
+<vertex x="61.3" y="43.1" curve="90"/>
+<vertex x="60.5" y="42.3"/>
+<vertex x="60.5" y="41.9"/>
+<vertex x="59.2" y="41.9"/>
+<vertex x="59.2" y="43.1"/>
+<vertex x="57.6" y="43.1"/>
 <vertex x="57.6" y="37.7"/>
+<vertex x="60.1" y="37.7"/>
+<vertex x="60.1" y="40.4"/>
+<vertex x="63.5" y="40.4"/>
+<vertex x="63.5" y="37.7"/>
 <vertex x="74.3" y="37.7"/>
 <vertex x="74.3" y="3.6"/>
 <vertex x="11.7" y="3.6"/>
 </polygon>
+<contactref element="B1" pad="1"/>
+<wire x1="61.15" y1="41.975" x2="61.603" y2="42.428" width="0.254" layer="1" curve="-90"/>
+<wire x1="61.603" y1="42.428" x2="64.911" y2="42.428" width="0.254" layer="1"/>
+<via x="62.4" y="39.9" extent="1-16" drill="0.254"/>
+<via x="63.8" y="37.1" extent="1-16" drill="0.254"/>
+<via x="62.4" y="38.5" extent="1-16" drill="0.254"/>
+<via x="62.4" y="37.1" extent="1-16" drill="0.254"/>
+<via x="65.2" y="37.1" extent="1-16" drill="0.254"/>
+<via x="66.6" y="37.1" extent="1-16" drill="0.254"/>
+<via x="68" y="37.1" extent="1-16" drill="0.254"/>
+<via x="69.4" y="37.1" extent="1-16" drill="0.254"/>
+<via x="70.8" y="37.1" extent="1-16" drill="0.254"/>
+<via x="72.2" y="37.1" extent="1-16" drill="0.254"/>
+<via x="73.6" y="37.1" extent="1-16" drill="0.254"/>
 </signal>
 <signal name="+3V3">
@@
 <contactref element="IC1" pad="25"/>
 <contactref element="B1" pad="4"/>
-<wire x1="58.35" y1="40.95" x2="59.325" y2="40.95" width="0.2032" layer="1"/>
-<wire x1="59.325" y1="40.95" x2="59.85" y2="40.425" width="0.2032" layer="1" curve="-90"/>
+<wire x1="58.35" y1="40.95" x2="59.325" y2="40.95" width="0.254" layer="1"/>
+<wire x1="59.325" y1="40.95" x2="59.85" y2="40.425" width="0.254" layer="1" curve="-90"/>
 </signal>
 <signal name="RFN">
 <contactref element="IC1" pad="26"/>
 <contactref element="B1" pad="3"/>
-<wire x1="58.35" y1="41.45" x2="59.325" y2="41.45" width="0.2032" layer="1"/>
-<wire x1="59.325" y1="41.45" x2="59.85" y2="41.975" width="0.2032" layer="1" curve="90"/>
+<wire x1="58.35" y1="41.45" x2="59.325" y2="41.45" width="0.254" layer="1"/>
+<wire x1="59.325" y1="41.45" x2="59.85" y2="41.975" width="0.254" layer="1" curve="90"/>
 </signal>
 <signal name="P0_3">
@@
 <wire x1="29.95" y1="56.75" x2="29.95" y2="52.5" width="0.254" layer="16"/>
 </signal>
-<signal name="N$6">
-<contactref element="R5" pad="1"/>
-<contactref element="B1" pad="1"/>
-<wire x1="62.25" y1="42.4" x2="61.575" y2="42.4" width="0.2032" layer="1"/>
-<wire x1="61.575" y1="42.4" x2="61.15" y2="41.975" width="0.2032" layer="1" curve="90"/>
-</signal>
 <signal name="N$2">
